File: projects/gate-controller/kicad/gate-controller/gate-controller.sch (KiCad schematic (older format))
At the start: 75 parts, among them U1 L7805, U2 Promini

Commit message: Gate controller
Parts:
- removed J_VCC: 6V, symbol Connector:Jack-DC
- removed J_VCC2: 12V, symbol Connector:Jack-DC
- added CN_D4, CN_D5, CN_D6, VM_D1: D, symbol Device:D
- added CN_Q4, CN_Q5: BC547, Package_TO_SOT_THT:TO-92_Inline, symbol Transistor_BJT:BC547
- added CN_R7, CN_R8: 10k, symbol Device:R
- added MO_K1, MO_K2: General_L3_K, symbol Own_Contractors:General_L3_K
- added MO_MOTOR: 3_Phase_Star_Shaped_Motor, symbol Own_Motors:3_Phase_Star_Shaped_Motor
- added MO_SW1: MO_SW1, symbol Own_Switches:SW_DPST_TRIPLE
- added VM_DPST1: 10A, symbol Own_Switches:SW_DPST_3_Temperature
- added VM_F1: 1A, symbol Device:Fuse
- added VM_F2: 1.5A, symbol Device:Fuse
- added VM_PS1: 5V, Converter_ACDC:Converter_ACDC_HiLink_HLK-PMxx, symbol Converter_ACDC:HLK-PM01
- added VM_PS2: 12V, Converter_ACDC:Converter_ACDC_HiLink_HLK-PMxx, symbol Converter_ACDC:HLK-PM01
- CN_Q1, CN_Q2, CN_Q3: value BC547 -> BC338
- CN_U2: symbol Own_Converters:XL6009 -> gate-controller-rescue:XL6009-Own_Converters
- CN_U_CLOSE, CN_U_MAIN, CN_U_OPEN: symbol Own_Contractors:RSM954N -> gate-controller-rescue:RSM954N-Own_Contractors
- RF_U1: renamed from RF_U_RX; symbol Own_Modules:RF_RX_433MHz -> gate-controller-rescue:RF_RX_433MHz-Own_Modules
- U2: symbol Own_Arduino:Promini -> gate-controller-rescue:Promini-Own_Arduino
- renumbered C1 to VM_C1, U1 to VM_U1
Connections:
- net labels added: L1, L11, L2, L21, L3, L31, N, PE
- net labels removed: P_D11, P_D13
- wire segments 206 -> 357
Other:
- note added: "BLOKADA MECHANICZNA"
- note added: "CN (OUTPUT)"
- note added: "CO (INPUT)"
- note added: "MI (OUTPUT)"
- note added: "MO (OUTPUT)"
- note added: "Motor - MO"
- note added: "OM (INPUT)"
- note added: "OM (OUTPUT)"
- note added: "RF (INPUT)"
- note added: "RF (OUTPUT)"
- note added: "VCC Module - VM"
- note added: "VM"
- note removed: "Contactors - CN"
- moved on the sheet: CN_D1, CN_D2, CN_D3, CN_J_CLOSE, CN_J_OPEN, CN_LED1, CN_LED2, CN_LED3, CN_Q1, CN_Q2, CN_Q3, CN_R1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

Commit message: Różne zmiany.
Parts:
- removed CN_U_CLOSE: RSM954N, symbol gate-controller-rescue:RSM954N-Own_Contractors
- removed CO_R12, CO_R15, CO_R2, CO_R5, CO_R9: 330, symbol Device:R
- added CN_U_CLOSE1: RSM954N, Own_Contractors:RSM954N, symbol gate-controller-rescue:RSM954N-Own_Contractors
- added VM_12V1, VM_5V1: Screw_Terminal_01x02, TerminalBlock:TerminalBlock_bornier-2_P5.08mm, symbol Connector:Screw_Terminal_01x02
- CN_D1, CN_D2, CN_D3, CN_D4, CN_D5, CN_D6, CN_LED1, CN_LED2, CN_LED3, CO_D1, CO_D2, CO_D3, CO_D4, CO_D5, MI_D1, MI_LED1, OM_D1, OM_LED1, RF_LED1: footprint (none) -> Diode_THT:D_5W_P5.08mm_Vertical_AnodeUp
- CN_J_CLOSE1: renamed from CN_J_CLOSE; footprint (none) -> TerminalBlock:TerminalBlock_bornier-2_P5.08mm
- CN_J_OPEN1: renamed from CN_J_OPEN; footprint (none) -> TerminalBlock:TerminalBlock_bornier-2_P5.08mm
- CN_Q1, CN_Q2, CN_Q3: footprint (none) -> Package_TO_SOT_THT:TO-92_Inline; symbol Device:Q_NPN_BCE -> Transistor_BJT:BC338
- CN_R1, CN_R3, CN_R5: value 330 -> 1k; footprint (none) -> Resistor_THT:R_Axial_DIN0204_L3.6mm_D1.6mm_P5.08mm_Horizontal
- CN_R2, CN_R4, CN_R6, CN_R7, CN_R8, CO_R1, CO_R10, CO_R11, CO_R13, CO_R14, CO_R3, CO_R4, CO_R6, CO_R7, CO_R9, MI_R1, MI_R2, OM_R1, OM_R2, RF_R1: footprint (none) -> Resistor_THT:R_Axial_DIN0204_L3.6mm_D1.6mm_P5.08mm_Horizontal
- CN_U2: footprint (none) -> Own_Modules:XL6009
- CN_U_MAIN1: renamed from CN_U_MAIN; footprint (none) -> Own_Contractors:RSM954N
- CN_U_OPEN1: renamed from CN_U_OPEN; footprint (none) -> Own_Contractors:RSM954N
- CO_C1, CO_C2, CO_C3, CO_C4, CO_C5, VM_C1: footprint (none) -> Capacitor_THT:CP_Radial_D5.0mm_P2.50mm
- CO_J_CLOSE1: renamed from CO_J_CLOSE; footprint (none) -> TerminalBlock:TerminalBlock_bornier-2_P5.08mm
- CO_J_LIMIT_CLOSE1: renamed from CO_J_LIMIT_CLOSE; footprint (none) -> TerminalBlock:TerminalBlock_bornier-2_P5.08mm
- CO_J_LIMIT_OPEN1: renamed from CO_J_LIMIT_OPEN; footprint (none) -> TerminalBlock:TerminalBlock_bornier-2_P5.08mm
- CO_J_OPEN1: renamed from CO_J_OPEN; footprint (none) -> TerminalBlock:TerminalBlock_bornier-2_P5.08mm
- CO_J_STOP1: renamed from CO_J_STOP; footprint (none) -> TerminalBlock:TerminalBlock_bornier-2_P5.08mm
- CO_SW_CLOSE1: renamed from CO_SW_CLOSE; footprint (none) -> Button_Switch_THT:SW_TH_Tactile_Omron_B3F-10xx
- CO_SW_LIMIT_CLOSE1: renamed from CO_SW_LIMIT_CLOSE; footprint (none) -> Button_Switch_THT:SW_TH_Tactile_Omron_B3F-10xx
- CO_SW_LIMIT_OPEN1: renamed from CO_SW_LIMIT_OPEN; footprint (none) -> Button_Switch_THT:SW_TH_Tactile_Omron_B3F-10xx
- CO_SW_OPEN1: renamed from CO_SW_OPEN; footprint (none) -> Button_Switch_THT:SW_TH_Tactile_Omron_B3F-10xx
- CO_SW_STOP1: renamed from CO_SW_STOP; footprint (none) -> Button_Switch_THT:SW_TH_Tactile_Omron_B3F-10xx
- MI_OUT1: renamed from MI_OUT; footprint (none) -> TerminalBlock:TerminalBlock_bornier-2_P5.08mm
- OM_J_SIGNAL1: renamed from OM_J_SIGNAL; footprint (none) -> TerminalBlock:TerminalBlock_bornier-2_P5.08mm
- OM_J_SWITCH1: renamed from OM_J_SWITCH; footprint (none) -> TerminalBlock:TerminalBlock_bornier-2_P5.08mm
- RF_U1: footprint (none) -> Own_Modules:RF_RX_433MHz
- U2: footprint (none) -> Own_Modules:Arduino_Pro_Mini
- VM_D1: value D -> 1N4148; footprint (none) -> Diode_THT:D_5W_P5.08mm_Vertical_AnodeUp
- VM_F1, VM_F2: footprint (none) -> Own_Other:Fuse_5X20
- VM_U1: footprint (none) -> Package_TO_SOT_THT:TO-220-3_Vertical
- renumbered MO_MOTOR to MO_MOTOR1
Connections:
- net GND: now also VM_5V1.1 (Pin_1); no longer VM_PS1.3 (-Vout)
- net GND2: now also VM_12V1.1 (Pin_1); no longer VM_PS2.3 (-Vout)
- net VCC: now also CN_U_CLOSE1.5 (2); no longer CO_D1.2 (A), CO_D2.2 (A), CO_D3.2 (A), CO_D4.2 (A), CO_D5.2 (A)
- net XL6009_OUT_+: now also CN_U_CLOSE1.1 (7)
- net at CN_D4.2 (A), CN_U_MAIN1.2 (11): now also CN_Q1.1 (C); no longer CN_Q1.2 (C)
- net at CN_R2.1: now also CN_Q1.2 (B); no longer CN_Q1.1 (B)
- net at CO_R1.1, CO_SW_CLOSE1.1 (A), CO_SW_CLOSE1.2 (A): now also CO_D1.2 (A)
- net at CO_R4.1, CO_SW_OPEN1.1 (A), CO_SW_OPEN1.2 (A): now also CO_D2.2 (A)
- net at CO_J_OPEN1.2 (Pin_2): now also CO_D2.1 (K)
- net at CN_Q4.1 (C), CN_R4.1: now also CN_Q2.2 (B); no longer CN_Q2.1 (B)
- net at CN_D5.2 (A): now also CN_Q2.1 (C), CN_U_CLOSE1.2 (11); no longer CN_Q2.2 (C)
- net at CN_D2.2 (A): now also CN_U_CLOSE1.4 (1)
- net at CO_J_CLOSE1.2 (Pin_2): now also CO_D1.1 (K)
- net at CO_R7.1, CO_SW_STOP1.1 (A), CO_SW_STOP1.2 (A): now also CO_D3.2 (A)
- net at CO_J_STOP1.2 (Pin_2): now also CO_D3.1 (K)
- net at CN_Q5.1 (C), CN_R6.1: now also CN_Q3.2 (B); no longer CN_Q3.1 (B)
- net at CN_D6.2 (A), CN_U_OPEN1.2 (11): now also CN_Q3.1 (C); no longer CN_Q3.2 (C)
- net at VM_PS1.4 (+Vout): no longer VM_F1.2
- net at CO_R10.1, CO_SW_LIMIT_CLOSE1.1 (A), CO_SW_LIMIT_CLOSE1.2 (A): now also CO_D4.2 (A)
- net at CO_J_LIMIT_CLOSE1.2 (Pin_2): now also CO_D4.1 (K)
- net at VM_PS2.4 (+Vout): no longer VM_F2.2
- net at CO_R13.1, CO_SW_LIMIT_OPEN1.1 (A), CO_SW_LIMIT_OPEN1.2 (A): now also CO_D5.2 (A)
- net at CO_J_LIMIT_OPEN1.2 (Pin_2): now also CO_D5.1 (K)
- new net: VM_5V1.2 (Pin_2), VM_F1.2
- new net: VM_12V1.2 (Pin_2), VM_F2.2
- new net: MO_K1.1 (2), MO_K2.1 (2), MO_SW1.5
- new net: MO_K1.2 (5), MO_K2.2 (5), MO_SW1.3
- new net: MO_K1.3 (6), MO_K2.3 (6), MO_SW1.1
Other:
- note removed: "VM"
- moved on the sheet: CN_D1, CN_D2, CN_D3, CN_D4, CN_D5, CN_D6, CN_J_CLOSE1, CN_J_OPEN1, CN_LED1, CN_LED2, CN_LED3, CN_Q4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
