File: kicad/notes/notes/notes.sch (KiCad schematic (older format))
At the start: 21 parts, among them Q1 Q_NPN_BCE, Q2 Q_NPN_BCE, Q3 Q_NPN_BCE, Q4 Q_PNP_BCE

Commit message: Increment.
Parts:
- added BT?: Battery_Cell, symbol Device:Battery_Cell
- added BZ12: Buzzer, symbol Device:Buzzer
- added C14: C, symbol Device:C
- added D1, D11, D7: LED, symbol Device:LED
- added F2: A1050, OptoDevice:R_LDR_D6.4mm_P3.4mm_Vertical, symbol Sensor_Optical:A1050
- added Q5, Q9: Q_NPN_BCE, symbol Device:Q_NPN_BCE
- added R10, R13, R3, R4, R6, R8: R, symbol Device:R
Connections:
- new net: BT?.1 (+), BZ12.1 (-), D1.2 (A), D11.2 (A), D7.2 (A)
- new net: BT?.2 (-), C14.2, Q5.3 (E), Q9.3 (E), R3.1
- new net: D1.1 (K), F2.1
- new net: D7.1 (K), R6.1
- new net: D11.1 (K), R10.1
- new net: Q5.2 (C), R6.2, R8.2
- new net: BZ12.2 (+), Q9.2 (C), R10.2, R13.1
- new net: Q5.1 (B), R13.2, R4.1
- new net: Q9.1 (B), R8.1
- new net: C14.1, F2.2, R3.2, R4.2
Other:
- moved on the sheet: BZ1, D1, D2, Q1, Q2, Q3, Q4, R1, R2, R3, R4

Commit message: Update
Parts:
- added BT?: Battery_Cell, symbol Device:Battery_Cell
- added D? (x2): 3.6V, symbol Device:D_Zener
- added R? (x2): 63, symbol Device:R
- added R?: 2k2, symbol Device:R
- added R?: 4k7, symbol Device:R
- added U?: ATtiny85-20MU, Package_DFN_QFN:QFN-20-1EP_4x4mm_P0.5mm_EP2.6x2.6mm, symbol MCU_Microchip_ATtiny:ATtiny85-20MU
Connections:
- new net: R?.1, U?.1 (~RESET~/PB5)
- new net: R?.2, U?.12 (PB1)
- new net: R?.2, U?.14 (PB2)
- new net: BT?.1 (+), R?.1, U?.15 (VCC)
- new net: BT?.2 (-), U?.21 (GND), U?.8 (GND)
- new net: D?.1 (K), R?.1
- new net: D?.1 (K), R?.1, R?.2
- new net +5V: R?.2
- new net GND: D?.2 (A), D?.2 (A)
Other:
- note added: "USB - D+ (green)"
- note added: "USB - D- (white)"
Changed lines of the file:
@@
 Wire Wire Line
 	6025 2500 6350 2500
+$Comp
+L MCU_Microchip_ATtiny:ATtiny85-20MU U?
+U 1 1 61EDC23D
+P 3150 3750
+F 0 "U?" H 2607 3796 50  0001 R CNN
+F 1 "ATtiny85-20MU" H 3300 3950 50  0000 R CNN
+F 2 "Package_DFN_QFN:QFN-20-1EP_4x4mm_P0.5mm_EP2.6x2.6mm" H 3150 3750 50  0001 C CIN
+F 3 "http://ww1.microchip.com/downloads/en/DeviceDoc/atmel-2586-avr-8-bit-microcontroller-attiny25-attiny45-attiny85_datasheet.pdf" H 3150 3750 50  0001 C CNN
+	1    3150 3750
+	1    0    0    -1
+$EndComp
+$Comp
+L Device:Battery_Cell BT?
+U 1 1 61EE30C6
+P 2000 3800
+F 0 "BT?" H 2118 3896 50  0001 L CNN
+F 1 "Battery_Cell" H 2100 3750 50  0001 L CNN
+F 2 "" V 2000 3860 50  0001 C CNN
+F 3 "~" V 2000 3860 50  0001 C CNN
+	1    2000 3800
+	1    0    0    -1
+$EndComp
+Wire Wire Line
+	3150 3050 3150 3150
+Wire Wire Line
+	3150 4450 3150 4350
+Wire Wire Line
+	2000 3900 2000 4450
+Wire Wire Line
+	2000 3600 2000 3050
+Wire Wire Line
+	2000 3050 3150 3050
+$Comp
+L Device:R R?
+U 1 1 61F0EB90
+P 4100 3550
+F 0 "R?" V 3900 3550 50  0001 C CNN
+F 1 "63" V 4000 3550 50  0000 C CNN
+F 2 "" V 4030 3550 50  0001 C CNN
+F 3 "~" H 4100 3550 50  0001 C CNN
+	1    4100 3550
+	0    1    1    0
+$EndComp
+Wire Wire Line
+	4250 3550 4400 3550
+$Comp
+L Device:D_Zener D?
+U 1 1 61F11FBF
+P 4400 3300
+F 0 "D?" V 4650 3550 50  0001 R CNN
+F 1 "3.6V" V 4550 3500 50  0000 R CNN
+F 2 "" H 4400 3300 50  0001 C CNN
+F 3 "~" H 4400 3300 50  0001 C CNN
+	1    4400 3300
+	0    -1   -1   0
+$EndComp
+Wire Wire Line
+	4400 3450 4400 3550
+Connection ~ 4400 3550
+$Comp
+L Device:R R?
+U 1 1 61F187B2
+P 4100 3650
+F 0 "R?" V 4300 3650 50  0001 C CNN
+F 1 "63" V 4200 3650 50  0000 C CNN
+F 2 "" V 4030 3650 50  0001 C CNN
+F 3 "~" H 4100 3650 50  0001 C CNN
+	1    4100 3650
+	0    1    1    0
+$EndComp
+Wire Wire Line
+	4250 3650 4850 3650
+Wire Wire Line
+	4400 3150 4400 2950
+$Comp
+L Device:D_Zener D?
+U 1 1 61F1F22B
+P 4850 3300
+F 0 "D?" V 5100 3550 50  0001 R CNN
+F 1 "3.6V" V 4950 3500 50  0000 R CNN
+F 2 "" H 4850 3300 50  0001 C CNN
+F 3 "~" H 4850 3300 50  0001 C CNN
+	1    4850 3300
+	0    -1   -1   0
+$EndComp
+Wire Wire Line
+	4850 3450 4850 3650
+Connection ~ 4850 3650
+$Comp
+L Device:R R?
+U 1 1 61F2275B
+P 5050 3300
+F 0 "R?" H 5120 3346 50  0001 L CNN
+F 1 "2k2" H 5120 3300 50  0000 L CNN
+F 2 "" V 4980 3300 50  0001 C CNN
+F 3 "~" H 5050 3300 50  0001 C CNN
+	1    5050 3300
+	1    0    0    -1
+$EndComp
+Wire Wire Line
+	4400 3550 5550 3550
+Wire Wire Line
+	4850 3650 5050 3650
+Wire Wire Line
+	5050 3450 5050 3650
+Connection ~ 5050 3650
+Wire Wire Line
+	5050 3650 5550 3650
+Wire Wire Line
+	4850 3150 4850 2950
+Wire Wire Line
+	4850 2950 4600 2950
+Wire Wire Line
+	4600 2950 4600 2750
+Connection ~ 4600 2950
+Wire Wire Line
+	4600 2950 4400 2950
+$Comp
+L power:GND #PWR?
+U 1 1 61F34D51
+P 4600 2750
+F 0 "#PWR?" H 4600 2500 50  0001 C CNN
+F 1 "GND" H 4605 2577 50  0000 C CNN
+F 2 "" H 4600 2750 50  0001 C CNN
+F 3 "" H 4600 2750 50  0001 C CNN
+	1    4600 2750
+	-1   0    0    1
+$EndComp
+Wire Wire Line
+	3150 3050 3150 2850
+Wire Wire Line
+	3150 2850 5050 2850
+Wire Wire Line
+	5050 2850 5050 3150
+Connection ~ 3150 3050
+Wire Wire Line
+	3750 3550 3950 3550
+Wire Wire Line
+	3750 3650 3950 3650
+Wire Wire Line
+	2000 4450 3150 4450
+$Comp
+L Device:R R?
+U 1 1 61F558A6
+P 3900 4150
+F 0 "R?" H 3970 4150 50  0001 L CNN
+F 1 "4k7" H 3970 4105 50  0001 L CNN
+F 2 "" V 3830 4150 50  0001 C CNN
+F 3 "~" H 3900 4150 50  0001 C CNN
+	1    3900 4150
+	1    0    0    -1
+$EndComp
+Wire Wire Line
+	3750 3950 3900 3950
+Wire Wire Line
+	3900 3950 3900 4000
+$Comp
+L power:+5V #PWR?
+U 1 1 61F5AC07
+P 3900 4300
+F 0 "#PWR?" H 3900 4150 50  0001 C CNN
+F 1 "+5V" H 3915 4473 50  0000 C CNN
+F 2 "" H 3900 4300 50  0001 C CNN
+F 3 "" H 3900 4300 50  0001 C CNN
+	1    3900 4300
+	-1   0    0    1
+$EndComp
+Text Notes 5350 3750 0    39   ~ 0
+USB - D- (white)
+Text Notes 5350 3500 0    39   ~ 0
+USB - D+ (green)
 $EndSCHEMATC

Commit message: Update
Parts:
- added C?: C, symbol Device:C
- added R? (x2): R, symbol Device:R
- added SW? (x3): SW_DPST_x2, symbol Switch:SW_DPST_x2
- added U? (x3): ATtiny4-MA, Package_DFN_QFN:DFN-8-1EP_2x2mm_P0.5mm_EP0.9x1.5mm, symbol MCU_Microchip_ATtiny:ATtiny4-MA
Connections:
- net +5V: now also SW?.1 (A), SW?.2 (B), U?.5 (PB0)
- net GND: now also R?.1, R?.1, SW?.2 (B)
- new net: SW?.1 (A), U?.5 (PB0)
- new net: R?.2, SW?.2 (B)
- new net: C?.1, C?.2, R?.2, SW?.1 (A), U?.5 (PB0)
Changed lines of the file:
@@
 Text Notes 5350 3500 0    39   ~ 0
 USB - D+ (green)
+$Comp
+L MCU_Microchip_ATtiny:ATtiny4-MA U?
+U 1 1 624A496C
+P 1700 5700
+F 0 "U?" H 1156 5746 50  0000 R CNN
+F 1 "ATtiny4-MA" H 1156 5655 50  0000 R CNN
+F 2 "Package_DFN_QFN:DFN-8-1EP_2x2mm_P0.5mm_EP0.9x1.5mm" H 1700 5700 50  0001 C CIN
+F 3 "http://ww1.microchip.com/downloads/en/DeviceDoc/Atmel-8127-AVR-8-bit-Microcontroller-ATtiny4-ATtiny5-ATtiny9-ATtiny10_Datasheet.pdf" H 1700 5700 50  0001 C CNN
+	1    1700 5700
+	1    0    0    -1
+$EndComp
+Wire Wire Line
+	2300 5400 2500 5400
+$Comp
+L Switch:SW_DPST_x2 SW?
+U 1 1 624A9389
+P 2700 5400
+F 0 "SW?" H 2700 5635 50  0001 C CNN
+F 1 "SW_DPST_x2" H 2700 5544 50  0001 C CNN
+F 2 "" H 2700 5400 50  0001 C CNN
+F 3 "~" H 2700 5400 50  0001 C CNN
+	1    2700 5400
+	1    0    0    -1
+$EndComp
+Wire Wire Line
+	2900 5400 3100 5400
+$Comp
+L power:GND #PWR?
+U 1 1 624ADE6D
+P 3100 5400
+F 0 "#PWR?" H 3100 5150 50  0001 C CNN
+F 1 "GND" V 3105 5272 50  0000 R CNN
+F 2 "" H 3100 5400 50  0001 C CNN
+F 3 "" H 3100 5400 50  0001 C CNN
+	1    3100 5400
+	0    -1   -1   0
+$EndComp
+$Comp
+L power:GND #PWR?
+U 1 1 624B7BAF
+P 3700 6750
+F 0 "#PWR?" H 3700 6500 50  0001 C CNN
+F 1 "GND" V 3705 6622 50  0000 R CNN
+F 2 "" H 3700 6750 50  0001 C CNN
+F 3 "" H 3700 6750 50  0001 C CNN
+	1    3700 6750
+	0    -1   -1   0
+$EndComp
+$Comp
+L Switch:SW_DPST_x2 SW?
+U 1 1 624B7BA8
+P 3000 6750
+F 0 "SW?" H 3000 6985 50  0001 C CNN
+F 1 "SW_DPST_x2" H 3000 6894 50  0001 C CNN
+F 2 "" H 3000 6750 50  0001 C CNN
+F 3 "~" H 3000 6750 50  0001 C CNN
+	1    3000 6750
+	1    0    0    -1
+$EndComp
+$Comp
+L MCU_Microchip_ATtiny:ATtiny4-MA U?
+U 1 1 624B7BA1
+P 1700 7050
+F 0 "U?" H 1156 7096 50  0000 R CNN
+F 1 "ATtiny4-MA" H 1156 7005 50  0000 R CNN
+F 2 "Package_DFN_QFN:DFN-8-1EP_2x2mm_P0.5mm_EP0.9x1.5mm" H 1700 7050 50  0001 C CIN
+F 3 "http://ww1.microchip.com/downloads/en/DeviceDoc/Atmel-8127-AVR-8-bit-Microcontroller-ATtiny4-ATtiny5-ATtiny9-ATtiny10_Datasheet.pdf" H 1700 7050 50  0001 C CNN
+	1    1700 7050
+	1    0    0    -1
+$EndComp
+Wire Wire Line
+	2300 6750 2550 6750
+$Comp
+L Device:R R?
+U 1 1 624D3A70
+P 3450 6750
+F 0 "R?" V 3243 6750 50  0001 C CNN
+F 1 "R" V 3334 6750 50  0001 C CNN
+F 2 "" V 3380 6750 50  0001 C CNN
+F 3 "~" H 3450 6750 50  0001 C CNN
+	1    3450 6750
+	0    1    1    0
+$EndComp
+Wire Wire Line
+	3200 6750 3300 6750
+Wire Wire Line
+	3600 6750 3700 6750
+Wire Wire Line
+	2550 6750 2550 6400
+Wire Wire Line
+	2550 6400 3650 6400
+Connection ~ 2550 6750
+Wire Wire Line
+	2550 6750 2800 6750
+$Comp
+L power:+5V #PWR?
+U 1 1 624E0702
+P 3650 6400
+F 0 "#PWR?" H 3650 6250 50  0001 C CNN
+F 1 "+5V" V 3665 6528 50  0000 L CNN
+F 2 "" H 3650 6400 50  0001 C CNN
+F 3 "" H 3650 6400 50  0001 C CNN
+	1    3650 6400
+	0    1    1    0
+$EndComp
+$Comp
+L Switch:SW_DPST_x2 SW?
+U 1 1 624E3D0F
+P 5950 5400
+F 0 "SW?" H 5950 5635 50  0001 C CNN
+F 1 "SW_DPST_x2" H 5950 5544 50  0001 C CNN
+F 2 "" H 5950 5400 50  0001 C CNN
+F 3 "~" H 5950 5400 50  0001 C CNN
+	1    5950 5400
+	1    0    0    -1
+$EndComp
+$Comp
+L MCU_Microchip_ATtiny:ATtiny4-MA U?
+U 1 1 624E3D15
+P 4650 5700
+F 0 "U?" H 4106 5746 50  0000 R CNN
+F 1 "ATtiny4-MA" H 4106 5655 50  0000 R CNN
+F 2 "Package_DFN_QFN:DFN-8-1EP_2x2mm_P0.5mm_EP0.9x1.5mm" H 4650 5700 50  0001 C CIN
+F 3 "http://ww1.microchip.com/downloads/en/DeviceDoc/Atmel-8127-AVR-8-bit-Microcontroller-ATtiny4-ATtiny5-ATtiny9-ATtiny10_Datasheet.pdf" H 4650 5700 50  0001 C CNN
+	1    4650 5700
+	1    0    0    -1
+$EndComp
+Wire Wire Line
+	5250 5400 5500 5400
+Wire Wire Line
+	5500 5400 5500 5050
+Wire Wire Line
+	5500 5050 5650 5050
+Connection ~ 5500 5400
+Wire Wire Line
+	5500 5400 5650 5400
+$Comp
+L power:+5V #PWR?
+U 1 1 624E3D28
+P 6650 5400
+F 0 "#PWR?" H 6650 5250 50  0001 C CNN
+F 1 "+5V" V 6665 5528 50  0000 L CNN
+F 2 "" H 6650 5400 50  0001 C CNN
+F 3 "" H 6650 5400 50  0001 C CNN
+	1    6650 5400
+	0    1    1    0
+$EndComp
+$Comp
+L power:GND #PWR?
+U 1 1 624E3D09
+P 6600 5050
+F 0 "#PWR?" H 6600 4800 50  0001 C CNN
+F 1 "GND" V 6605 4922 50  0000 R CNN
+F 2 "" H 6600 5050 50  0001 C CNN
+F 3 "" H 6600 5050 50  0001 C CNN
+	1    6600 5050
+	0    -1   -1   0
+$EndComp
+Wire Wire Line
+	6150 5400 6650 5400
+$Comp
+L Device:C C?
+U 1 1 624F5E37
+P 5650 5200
+F 0 "C?" H 5765 5246 50  0001 L CNN
+F 1 "C" H 5765 5155 50  0001 L CNN
+F 2 "" H 5688 5050 50  0001 C CNN
+F 3 "~" H 5650 5200 50  0001 C CNN
+	1    5650 5200
+	1    0    0    -1
+$EndComp
+Connection ~ 5650 5050
+Wire Wire Line
+	5650 5350 5650 5400
+Connection ~ 5650 5400
+Wire Wire Line
+	5650 5400 5750 5400
+Wire Wire Line
+	5650 5050 5850 5050
+Wire Wire Line
+	6150 5050 6600 5050
+$Comp
+L Device:R R?
+U 1 1 624E3D1C
+P 6000 5050
+F 0 "R?" V 5793 5050 50  0001 C CNN
+F 1 "R" V 5884 5050 50  0001 C CNN
+F 2 "" V 5930 5050 50  0001 C CNN
+F 3 "~" H 6000 5050 50  0001 C CNN
+	1    6000 5050
+	0    1    1    0
+$EndComp
 $EndSCHEMATC
